File: Full_Bridge_Rectifier/Full_Bridge_Rectifier.kicad_sch (KiCad schematic)
At the start: 9 parts, among them J1 Conn_01x02_Socket, J2 Conn_01x02_Socket

Commit message: 2EI4 lab1 complete
Parts:
- C1, C2: footprint (none) -> Capacitor_THT:CP_Radial_D4.0mm_P2.00mm
Changed lines of the file:
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@@
 			)
 		)
-		(property "Footprint" ""
+		(property "Footprint" "Capacitor_THT:CP_Radial_D4.0mm_P2.00mm"
 			(at 157.48 102.87 0)
 			(effects
@@
 			)
 		)
-		(property "Footprint" ""
+		(property "Footprint" "Capacitor_THT:CP_Radial_D4.0mm_P2.00mm"
 			(at 163.83 102.87 0)
 			(effects
@@
 		)
 	)
+	(sheet_instances
+		(path "/"
+			(page "1")
+		)
+	)
+	(embedded_fonts no)
 )
