File: MOSFET_Switch/MOSFET_Switch.kicad_sch (KiCad schematic)
At the start: 0 parts

Commit message: update
Parts:
- added J1, J2: Conn_01x02_Pin, Connector_PinHeader_2.00mm:PinHeader_1x02_P2.00mm_Vertical, symbol Connector:Conn_01x02_Pin
- added U1: ~, Package_DIP:DIP-14_W7.62mm, symbol Transistor_FET:CD4007
