File: FullBridgeRectifier/Full_Bridge_Rectifier.kicad_pcb (KiCad board)
At the start: 2 copper layers, 9 parts, among them J1 Conn_01x02_Socket, J2 Conn_01x02_Socket

Commit message: update
Other:
- board outline added: 35.5 x 24.5 mm
Changed lines of the file:
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@@
 		)
 	)
-	(gr_line
-		(start 169.5 113.5)
-		(end 169.5 89)
+	(gr_rect
+		(start 134 89)
+		(end 169.5 113.5)
 		(stroke
-			(width 0.2)
+			(width 0.05)
 			(type default)
 		)
-		(layer "F.Cu")
-	)
-	(gr_line
-		(start 134 89)
-		(end 134 112.5)
-		(stroke
-			(width 0.2)
-			(type default)
-		)
-		(layer "F.Cu")
-	)
-	(gr_line
-		(start 134 113.5)
-		(end 169 113.5)
-		(stroke
-			(width 0.2)
-			(type default)
-		)
-		(layer "F.Cu")
-	)
-	(gr_line
-		(start 169 113.5)
-		(end 169.5 113.5)
-		(stroke
-			(width 0.2)
-			(type default)
-		)
-		(layer "F.Cu")
-	)
-	(gr_line
-		(start 134 112.5)
-		(end 134 113.5)
-		(stroke
-			(width 0.2)
-			(type default)
-		)
-		(layer "F.Cu")
-	)
-	(gr_line
-		(start 169.5 89)
-		(end 134 89)
-		(stroke
-			(width 0.2)
-			(type default)
-		)
-		(layer "F.Cu")
+		(fill no)
+		(layer "Edge.Cuts")
 	)
 	(gr_text "+"
