File: XORgate/XORgate.kicad_pcb (KiCad board)
At the start: 2 copper layers, 6 parts, among them J1 Conn_01x02_Pin, J2 Conn_01x02_Pin, J3 Conn_01x02_Pin, J4 Conn_01x02_Pin

Commit message: update
Connections:
- net Net-(J1-Pin_1) renamed A
- net Net-(J2-Pin_1) renamed B
- net Net-(J4-Pin_1) renamed Vcc
- net Net-(U1C-D) renamed A'
- net Net-(U1E-G) renamed B'
Changed lines of the file:
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@@
 	(net 0 "")
 	(net 1 "GND")
-	(net 2 "Net-(J1-Pin_1)")
-	(net 3 "Net-(J2-Pin_1)")
+	(net 2 "A")
+	(net 3 "B")
 	(net 4 "Net-(J3-Pin_1)")
-	(net 5 "Net-(J4-Pin_1)")
+	(net 5 "Vcc")
 	(net 6 "Net-(U1B-D)")
 	(net 7 "Net-(U1B-S)")
 	(net 8 "Net-(U1A-S)")
 	(net 9 "Net-(U1A-D)")
-	(net 10 "Net-(U1C-D)")
+	(net 10 "A'")
 	(net 11 "Net-(U2A-S)")
-	(net 12 "Net-(U1E-G)")
+	(net 12 "B'")
 	(net 13 "Net-(U1D-S)")
 	(footprint "Connector_PinHeader_2.00mm:PinHeader_1x02_P2.00mm_Vertical"
@@
 			(layers "*.Cu" "*.Mask")
 			(remove_unused_layers no)
-			(net 2 "Net-(J1-Pin_1)")
+			(net 2 "A")
 			(pinfunction "Pin_1")
 			(pintype "passive")
@@
 			(layers "*.Cu" "*.Mask")
 			(remove_unused_layers no)
-			(net 2 "Net-(J1-Pin_1)")
+			(net 2 "A")
 			(pinfunction "G")
 			(pintype "input")
@@
 			(layers "*.Cu" "*.Mask")
 			(remove_unused_layers no)
-			(net 2 "Net-(J1-Pin_1)")
+			(net 2 "A")
 			(pinfunction "G")
 			(pintype "input")
@@
 			(layers "*.Cu" "*.Mask")
 			(remove_unused_layers no)
-			(net 10 "Net-(U1C-D)")
+			(net 10 "A'")
 			(pinfunction "D")
 			(pintype "passive")
@@
 			(layers "*.Cu" "*.Mask")
 			(remove_unused_layers no)
-			(net 10 "Net-(U1C-D)")
+			(net 10 "A'")
 			(pinfunction "G")
 			(pintype "input")
@@
 			(layers "*.Cu" "*.Mask")
 			(remove_unused_layers no)
-			(net 10 "Net-(U1C-D)")
+			(net 10 "A'")
 			(pinfunction "S")
 			(pintype "passive")
@@
 			(layers "*.Cu" "*.Mask")
 			(remove_unused_layers no)
-			(net 5 "Net-(J4-Pin_1)")
+			(net 5 "Vcc")
 			(pinfunction "D")
 			(pintype "passive")
@@
 			(layers "*.Cu" "*.Mask")
 			(remove_unused_layers no)
-			(net 5 "Net-(J4-Pin_1)")
+			(net 5 "Vcc")
 			(pinfunction "Pin_1")
 			(pintype "passive")
@@
 			(layers "*.Cu" "*.Mask")
 			(remove_unused_layers no)
-			(net 10 "Net-(U1C-D)")
+			(net 10 "A'")
 			(pinfunction "G")
 			(pintype "input")
@@
 			(layers "*.Cu" "*.Mask")
 			(remove_unused_layers no)
-			(net 3 "Net-(J2-Pin_1)")
+			(net 3 "B")
 			(pinfunction "G")
 			(pintype "input")
@@
 			(layers "*.Cu" "*.Mask")
 			(remove_unused_layers no)
-			(net 12 "Net-(U1E-G)")
+			(net 12 "B'")
 			(pinfunction "D")
 			(pintype "passive")
@@
 			(layers "*.Cu" "*.Mask")
 			(remove_unused_layers no)
-			(net 3 "Net-(J2-Pin_1)")
+			(net 3 "B")
 			(pinfunction "G")
 			(pintype "input")
@@
 			(layers "*.Cu" "*.Mask")
 			(remove_unused_layers no)
-			(net 12 "Net-(U1E-G)")
+			(net 12 "B'")
 			(pinfunction "S")
 			(pintype "passive")
@@
 			(layers "*.Cu" "*.Mask")
 			(remove_unused_layers no)
-			(net 5 "Net-(J4-Pin_1)")
+			(net 5 "Vcc")
 			(pinfunction "D")
 			(pintype "passive")
@@
 			(layers "*.Cu" "*.Mask")
 			(remove_unused_layers no)
-			(net 3 "Net-(J2-Pin_1)")
+			(net 3 "B")
 			(pinfunction "Pin_1")
 			(pintype "passive")

Commit message: XOR gate
Parts:
- added J5: Conn_01x02_Pin, Connector_PinHeader_2.00mm:PinHeader_1x02_P2.00mm_Vertical, F.Cu at (191.5, 80.0)
- added J6: Conn_01x02_Pin, Connector_PinHeader_2.00mm:PinHeader_1x02_P2.00mm_Vertical, F.Cu at (191.5, 83.0)
- moved J4 82.2 mm to (141.5, 86.0), turned to 90 degrees
- moved J2 77.7 mm to (141.5, 83.0), turned to 90 degrees
- moved J1 76.8 mm to (141.5, 80.0), turned to 90 degrees
- moved J3 49.9 mm to (191.5, 86.0), turned to 90 degrees
- moved U2 9.83 mm to (172.9, 81.5)
- moved U1 9.39 mm to (154.4, 81.5)
Connections:
- U1 pad 2: Net-(U1A-D) -> Vcc
- U1 pad 4: Net-(U1B-S) -> GND
- U2 pad 2: Net-(U1A-D) -> Vcc
- U2 pad 4: Net-(U1B-S) -> GND
Routing:
- net Vcc: track 0.00 -> 156.7 mm
- net B: track 0.00 -> 155.1 mm
- net A: track 0.00 -> 75.3 mm
- net Net-(J3-Pin_1): track 0.00 -> 66.8 mm
- net A': track 0.00 -> 65.3 mm
- net Net-(U1A-S): track 0.00 -> 44.2 mm
- net B': track 0.00 -> 29.5 mm
- net Net-(U2A-S): track 0.00 -> 21.2 mm
- added copper zone on B.Cu, net GND
- added copper zone on F.Cu, net GND
- added copper zone on In1.Cu, net GND
- added copper zone on In2.Cu, net GND
Other:
- board outline added: 62.5 x 24 mm
- copper layers 2 -> 4
- board text added: "+"
- board text added: "A"
- board text added: "A'"
- board text added: "B"
- board text added: "B'"
- board text added: "GND"
- board text added: "Output"
- board text added: "Vcc"
